Commit message: trajectory added

File: rsc/wheelyBot.urdf (robot description, URDF)
Before this commit: robot wheelyBot, 7 links, 6 joints
Links:
- link Shank_L: mass 0.4 -> 4; geometry collision box size=0.06 0.020 0.254; visual box size=0.06 0.020 0.254
- link Shank_R: mass 0.4 -> 4; geometry collision box size=0.06 0.020 0.254; visual box size=0.06 0.020 0.254
- link Thigh_L: mass 0.4 -> 4; geometry collision box size=0.06 0.020 0.23728; visual box size=0.06 0.020 0.23728
- link Thigh_R: mass 0.4 -> 4; geometry collision box size=0.06 0.020 0.23728; visual box size=0.06 0.020 0.23728
- link Wheel_L: mass 0.530 -> 1.5; geometry collision cylinder length=0.05 radius=0.254; visual cylinder length=0.05 radius=0.254
- link Wheel_R: mass 0.530 -> 1.5; geometry collision cylinder length=0.05 radius=0.254; visual cylinder length=0.05 radius=0.254
- link torso: mass 5 -> 12
Joints:
- joint Knee_FE_L: origin xyz=0 0.02 -0.250 rpy=0 0 0 -> xyz=0 0.02 -0.23728 rpy=0 0 0
- joint Knee_FE_R: origin xyz=0 -0.02 -0.250 rpy=0 0 0 -> xyz=0 -0.02 -0.23728 rpy=0 0 0
- joint Wheel_Joint_L: origin xyz=0 0.0225 -0.250 rpy=0 0 0 -> xyz=0 0.0225 -0.254 rpy=0 0 0
- joint Wheel_Joint_R: origin xyz=0 -0.0225 -0.250 rpy=0 0 0 -> xyz=0 -0.0225 -0.254 rpy=0 0 0
